File: schaltplan/MicTonpegel.brd (EAGLE design)
At the start: 100 x 80 mm, 8 parts, among them IC1 MEGA16-A, M1 ELECTRET_MICROPHON-F6035AP, T1 2N3904

Commit message: Changed to actual wiring
Parts:
- removed B1: (no value), rectifier:B-DIL
- removed R2, R3: 10k, resistor:0207/2V
- removed T1: 2N3904, transistor:TO92
- R1: value 100k -> 2,2k
- moved R1 19.9 mm to (-16.5, 43.2)
Connections:
- removed net N$4: C1.1, R1.2, T1.2
- removed net N$5: B1.+, IC1.30
- removed net VCC: IC1.5
- net GND: no longer B1.-, B1.AC2, T1.3
- net N$1: now also IC1.5, R1.2; no longer C1.2, M1.1, R3.2
- net N$2: now also C1.1, M1.1, R1.1; no longer R2.1, R3.1
- net N$3: now also C1.2, IC1.37; no longer B1.AC1, R1.1, R2.2, T1.1
Changed lines of the file:
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@@
 <?xml version="1.0" encoding="utf-8"?>
 <!DOCTYPE eagle SYSTEM "eagle.dtd">
-<eagle version="6.2">
+<eagle version="6.0">
 <drawing>
 <settings>
@@
 <attribute name="OC_FARNELL" value="9171134" x="0" y="0" size="1.778" layer="27" display="off"/>
 </element>
-<element name="R1" library="resistor" package="0207/2V" value="100k" x="-34.29" y="34.29"/>
-<element name="R2" library="resistor" package="0207/2V" value="10k" x="-40.64" y="34.29"/>
-<element name="R3" library="resistor" package="0207/2V" value="10k" x="-16.51" y="43.18"/>
+<element name="R1" library="resistor" package="0207/2V" value="2,2k" x="-16.51" y="43.18"/>
 <element name="M1" library="microphon" package="F6035AP" value="ELECTRET_MICROPHON-F6035AP" x="-41.91" y="25.4"/>
 <element name="C1" library="capacitor-wima" package="C2.5-3" value="0,1µF" x="-26.67" y="34.29"/>
-<element name="T1" library="transistor" package="TO92" value="2N3904" x="-29.21" y="43.18"/>
-<element name="B1" library="rectifier" package="B-DIL" value="" x="-17.78" y="35.56"/>
 </elements>
 <signals>
 <signal name="GND">
 <contactref element="IC1" pad="28"/>
-<contactref element="M1" pad="2"/>
-<contactref element="T1" pad="3"/>
-<contactref element="B1" pad="AC2"/>
-<contactref element="B1" pad="-"/>
 <contactref element="IC1" pad="6"/>
 <contactref element="IC1" pad="6"/>
-<wire x1="-28.66" y1="10.16" x2="-41.91" y2="24.45" width="0" layer="19" extent="1-1"/>
+<contactref element="M1" pad="2"/>
 <wire x1="-17.06" y1="10.16" x2="-28.66" y2="10.16" width="0" layer="19" extent="1-1"/>
-<wire x1="-15.24" y1="31.75" x2="-17.06" y2="10.16" width="0" layer="19" extent="1-1"/>
-<wire x1="-20.32" y1="39.37" x2="-15.24" y2="31.75" width="0" layer="19" extent="1-1"/>
-<wire x1="-30.48" y1="43.18" x2="-20.32" y2="39.37" width="0" layer="19" extent="1-1"/>
+<wire x1="-41.91" y1="24.45" x2="-28.66" y2="10.16" width="0" layer="19" extent="1-1"/>
 </signal>
 <signal name="AVCC">
@@
 <contactref element="IC1" pad="17"/>
 </signal>
-<signal name="VCC">
-<contactref element="IC1" pad="5"/>
-</signal>
 <signal name="VCC2">
 <contactref element="IC1" pad="38"/>
 </signal>
 <signal name="N$1">
+<contactref element="IC1" pad="5"/>
+<contactref element="R1" pad="2"/>
+<wire x1="-28.66" y1="10.96" x2="-15.24" y2="43.18" width="0" layer="19" extent="1-1"/>
+</signal>
+<signal name="N$2">
+<contactref element="R1" pad="1"/>
 <contactref element="M1" pad="1"/>
-<contactref element="R3" pad="2"/>
+<contactref element="C1" pad="1"/>
+<wire x1="-27.94" y1="34.29" x2="-17.78" y2="43.18" width="0" layer="19" extent="1-1"/>
+<wire x1="-41.91" y1="26.35" x2="-27.94" y2="34.29" width="0" layer="19" extent="1-1"/>
+</signal>
+<signal name="N$3">
 <contactref element="C1" pad="2"/>
-<wire x1="-25.4" y1="34.29" x2="-15.24" y2="43.18" width="0" layer="19" extent="1-1"/>
-<wire x1="-41.91" y1="26.35" x2="-25.4" y2="34.29" width="0" layer="19" extent="1-1"/>
-</signal>
-<signal name="N$2">
-<contactref element="R3" pad="1"/>
-<contactref element="R2" pad="1"/>
-<wire x1="-41.91" y1="34.29" x2="-17.78" y2="43.18" width="0" layer="19" extent="1-1"/>
-</signal>
-<signal name="N$3">
-<contactref element="R2" pad="2"/>
-<contactref element="T1" pad="1"/>
-<contactref element="R1" pad="1"/>
-<contactref element="B1" pad="AC1"/>
-<wire x1="-27.94" y1="43.18" x2="-15.24" y2="39.37" width="0" layer="19" extent="1-1"/>
-<wire x1="-35.56" y1="34.29" x2="-27.94" y2="43.18" width="0" layer="19" extent="1-1"/>
-<wire x1="-39.37" y1="34.29" x2="-35.56" y2="34.29" width="0" layer="19" extent="1-1"/>
-</signal>
-<signal name="N$4">
-<contactref element="C1" pad="1"/>
-<contactref element="T1" pad="2"/>
-<contactref element="R1" pad="2"/>
-<wire x1="-27.94" y1="34.29" x2="-29.21" y2="45.085" width="0" layer="19" extent="1-1"/>
-<wire x1="-33.02" y1="34.29" x2="-27.94" y2="34.29" width="0" layer="19" extent="1-1"/>
-</signal>
-<signal name="N$5">
-<contactref element="B1" pad="+"/>
-<contactref element="IC1" pad="30"/>
-<wire x1="-17.06" y1="11.76" x2="-20.32" y2="31.75" width="0" layer="19" extent="1-1"/>
+<contactref element="IC1" pad="37"/>
+<wire x1="-21.26" y1="15.96" x2="-25.4" y2="34.29" width="0" layer="19" extent="1-1"/>
 </signal>
 </signals>
