File: schaltplan/MicTonpegel.sch (EAGLE design)
At the start: 8 parts, among them IC1 MEGA16-A, M1 ELECTRET_MICROPHON-F6035AP, T1 2N3904

Commit message: Changed to actual wiring
Parts:
- removed B1: (no value), rectifier:B-DIL
- removed R2, R3: 10k, resistor:R-EU_0207/2V
- removed T1: 2N3904, transistor:2N3904
- C1: value 0,1µF -> 0,1ÂµF
- R1: value 100k -> 2,2k
Connections:
- removed net N$4: C1.1, R1.2, T1.B
- removed net N$5: B1.+, IC1.(ADC7)PA7
- net GND: no longer B1.-, B1.AC2, T1.E
- net N$1: now also IC1.VCC, R1.2; no longer C1.2, M1.1, R3.2
- net N$2: now also C1.1, M1.1, R1.1; no longer R2.1, R3.1
- net N$3: now also C1.2, IC1.(ADC0)PA0; no longer B1.AC1, R1.1, R2.2, T1.C
Other:
- moved on the sheet: C1, R1
Changed lines of the file:
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@@
 <?xml version="1.0" encoding="utf-8"?>
 <!DOCTYPE eagle SYSTEM "eagle.dtd">
-<eagle version="6.2">
+<eagle version="6.0">
 <drawing>
 <settings>
@@
 <parts>
 <part name="IC1" library="atmel" deviceset="MEGA16" device="-A"/>
-<part name="R1" library="resistor" deviceset="R-EU_" device="0207/2V" value="100k"/>
-<part name="R2" library="resistor" deviceset="R-EU_" device="0207/2V" value="10k"/>
-<part name="R3" library="resistor" deviceset="R-EU_" device="0207/2V" value="10k"/>
+<part name="R1" library="resistor" deviceset="R-EU_" device="0207/2V" value="2,2k"/>
 <part name="M1" library="microphon" deviceset="ELECTRET_MICROPHON-" device="F6035AP"/>
-<part name="C1" library="capacitor-wima" deviceset="C" device="2,5-3" value="0,1µF"/>
-<part name="T1" library="transistor" deviceset="2N3904" device=""/>
+<part name="C1" library="capacitor-wima" deviceset="C" device="2,5-3" value="0,1ÂµF"/>
+<part name="GND2" library="supply1" deviceset="GND" device=""/>
 <part name="GND1" library="supply1" deviceset="GND" device=""/>
-<part name="B1" library="rectifier" deviceset="B-DIL" device=""/>
-<part name="GND2" library="supply1" deviceset="GND" device=""/>
 </parts>
 <sheets>
@@
 <instances>
 <instance part="IC1" gate="G$1" x="40.64" y="43.18"/>
-<instance part="R1" gate="G$1" x="116.84" y="83.82"/>
-<instance part="R2" gate="G$1" x="104.14" y="91.44" rot="R270"/>
-<instance part="R3" gate="G$1" x="157.48" y="91.44" rot="R270"/>
-<instance part="M1" gate="G$1" x="162.56" y="63.5"/>
-<instance part="C1" gate="G$1" x="134.62" y="68.58" rot="R90"/>
-<instance part="T1" gate="G1" x="106.68" y="68.58" rot="MR0"/>
-<instance part="GND1" gate="1" x="104.14" y="43.18"/>
-<instance part="B1" gate="1" x="83.82" y="78.74"/>
+<instance part="R1" gate="G$1" x="81.28" y="86.36" rot="R90"/>
+<instance part="M1" gate="G$1" x="91.44" y="68.58"/>
+<instance part="C1" gate="G$1" x="71.12" y="68.58" rot="R270"/>
 <instance part="GND2" gate="1" x="5.08" y="40.64"/>
+<instance part="GND1" gate="1" x="86.36" y="58.42"/>
 </instances>
 <busses>
@@
 <net name="GND" class="0">
 <segment>
-<pinref part="GND1" gate="1" pin="GND"/>
-<pinref part="M1" gate="G$1" pin="2"/>
-<wire x1="104.14" y1="45.72" x2="157.48" y2="45.72" width="0.1524" layer="91"/>
-<wire x1="157.48" y1="45.72" x2="157.48" y2="60.96" width="0.1524" layer="91"/>
-<pinref part="T1" gate="G1" pin="E"/>
-<wire x1="104.14" y1="63.5" x2="104.14" y2="45.72" width="0.1524" layer="91"/>
-<junction x="104.14" y="45.72"/>
-<pinref part="B1" gate="1" pin="AC2"/>
-<wire x1="83.82" y1="73.66" x2="83.82" y2="45.72" width="0.1524" layer="91"/>
-<wire x1="83.82" y1="45.72" x2="104.14" y2="45.72" width="0.1524" layer="91"/>
-<pinref part="B1" gate="1" pin="-"/>
-<wire x1="78.74" y1="78.74" x2="78.74" y2="45.72" width="0.1524" layer="91"/>
-<wire x1="78.74" y1="45.72" x2="83.82" y2="45.72" width="0.1524" layer="91"/>
-<junction x="83.82" y="45.72"/>
-</segment>
-<segment>
 <pinref part="IC1" gate="G$1" pin="GND"/>
 <wire x1="20.32" y1="45.72" x2="5.08" y2="45.72" width="0.1524" layer="91"/>
@@
 <wire x1="5.08" y1="45.72" x2="5.08" y2="43.18" width="0.1524" layer="91"/>
 </segment>
+<segment>
+<pinref part="M1" gate="G$1" pin="2"/>
+<pinref part="GND1" gate="1" pin="GND"/>
+<wire x1="86.36" y1="66.04" x2="86.36" y2="60.96" width="0.1524" layer="91"/>
+</segment>
 </net>
 <net name="N$1" class="0">
 <segment>
-<pinref part="M1" gate="G$1" pin="1"/>
-<pinref part="R3" gate="G$1" pin="2"/>
-<wire x1="157.48" y1="63.5" x2="157.48" y2="68.58" width="0.1524" layer="91"/>
-<pinref part="C1" gate="G$1" pin="2"/>
-<wire x1="157.48" y1="68.58" x2="157.48" y2="86.36" width="0.1524" layer="91"/>
-<wire x1="139.7" y1="68.58" x2="157.48" y2="68.58" width="0.1524" layer="91"/>
-<junction x="157.48" y="68.58"/>
+<pinref part="IC1" gate="G$1" pin="VCC"/>
+<wire x1="20.32" y1="55.88" x2="10.16" y2="55.88" width="0.1524" layer="91"/>
+<wire x1="10.16" y1="55.88" x2="10.16" y2="99.06" width="0.1524" layer="91"/>
+<wire x1="10.16" y1="99.06" x2="81.28" y2="99.06" width="0.1524" layer="91"/>
+<pinref part="R1" gate="G$1" pin="2"/>
+<wire x1="81.28" y1="99.06" x2="81.28" y2="91.44" width="0.1524" layer="91"/>
 </segment>
 </net>
 <net name="N$2" class="0">
 <segment>
-<pinref part="R3" gate="G$1" pin="1"/>
-<wire x1="157.48" y1="96.52" x2="157.48" y2="99.06" width="0.1524" layer="91"/>
-<wire x1="157.48" y1="99.06" x2="104.14" y2="99.06" width="0.1524" layer="91"/>
-<wire x1="104.14" y1="99.06" x2="104.14" y2="96.52" width="0.1524" layer="91"/>
-<pinref part="R2" gate="G$1" pin="1"/>
+<pinref part="R1" gate="G$1" pin="1"/>
+<pinref part="M1" gate="G$1" pin="1"/>
+<wire x1="81.28" y1="81.28" x2="81.28" y2="68.58" width="0.1524" layer="91"/>
+<wire x1="81.28" y1="68.58" x2="86.36" y2="68.58" width="0.1524" layer="91"/>
+<pinref part="C1" gate="G$1" pin="1"/>
+<wire x1="81.28" y1="68.58" x2="73.66" y2="68.58" width="0.1524" layer="91"/>
+<junction x="81.28" y="68.58"/>
 </segment>
 </net>
 <net name="N$3" class="0">
 <segment>
-<pinref part="R2" gate="G$1" pin="2"/>
-<pinref part="T1" gate="G1" pin="C"/>
-<wire x1="104.14" y1="86.36" x2="104.14" y2="83.82" width="0.1524" layer="91"/>
-<pinref part="R1" gate="G$1" pin="1"/>
-<wire x1="104.14" y1="83.82" x2="104.14" y2="73.66" width="0.1524" layer="91"/>
-<wire x1="111.76" y1="83.82" x2="104.14" y2="83.82" width="0.1524" layer="91"/>
-<junction x="104.14" y="83.82"/>
-<pinref part="B1" gate="1" pin="AC1"/>
-<wire x1="83.82" y1="83.82" x2="104.14" y2="83.82" width="0.1524" layer="91"/>
+<pinref part="C1" gate="G$1" pin="2"/>
+<pinref part="IC1" gate="G$1" pin="(ADC0)PA0"/>
+<wire x1="66.04" y1="68.58" x2="76.2" y2="68.58" width="0.1524" layer="91"/>
+<wire x1="66.04" y1="68.58" x2="60.96" y2="68.58" width="0.1524" layer="91"/>
 </segment>
 </net>
-<net name="N$4" class="0">
-<segment>
-<pinref part="C1" gate="G$1" pin="1"/>
-<pinref part="T1" gate="G1" pin="B"/>
-<wire x1="132.08" y1="68.58" x2="127" y2="68.58" width="0.1524" layer="91"/>
-<wire x1="127" y1="68.58" x2="109.22" y2="68.58" width="0.1524" layer="91"/>
-<pinref part="R1" gate="G$1" pin="2"/>
-<wire x1="121.92" y1="83.82" x2="127" y2="83.82" width="0.1524" layer="91"/>
-<wire x1="127" y1="83.82" x2="127" y2="68.58" width="0.1524" layer="91"/>
-<junction x="127" y="68.58"/>
-</segment>
-</net>
-<net name="N$5" class="0">
-<segment>
-<pinref part="B1" gate="1" pin="+"/>
-<wire x1="88.9" y1="78.74" x2="88.9" y2="86.36" width="0.1524" layer="91"/>
-<wire x1="88.9" y1="86.36" x2="60.96" y2="86.36" width="0.1524" layer="91"/>
-<pinref part="IC1" gate="G$1" pin="(ADC7)PA7"/>
-</segment>
-</net>
